File: Exterior.sch (KiCad schematic (older format))
At the start: 10 parts

Commit message: Generate PDFs
I opened this in the 4.0.2 version of kicad and it asked to make these changes.
Also included is the PDFs of the schematics.
Parts:
- A?: symbol ARGO -> Argo
- Aq?: symbol AQUASTAT -> Aquastat
- Grundfos, Taco: symbol CIRCULATOR -> Circulator
Changed lines of the file:
@@
-EESchema Schematic File Version 2  date Fri 20 Jun 2014 06:55:50 PM EDT
+EESchema Schematic File Version 2
+LIBS:Exterior-rescue
 LIBS:power
 LIBS:device
@@
 LIBS:memory
 LIBS:xilinx
-LIBS:special
 LIBS:microcontrollers
 LIBS:dsp
@@
 LIBS:boiler
 LIBS:relay
-EELAYER 25  0
+EELAYER 25 0
 EELAYER END
-$Descr A4 11700 8267
+$Descr A4 11693 8268
 encoding utf-8
 Sheet 1 1
@@
 Wire Wire Line
 	4450 5850 4550 5850
-Connection ~ 4450 3300
 Wire Wire Line
 	4450 5650 4550 5650
@@
 Wire Wire Line
 	4550 2400 4550 3400
-Connection ~ 4550 3400
 Wire Wire Line
 	2300 2700 2300 2800
@@
 F 0 "#PWR?" H 2950 6300 30  0001 C CNN
 F 1 "GND" H 2950 6230 30  0001 C CNN
+F 2 "" H 2950 6300 60  0001 C CNN
+F 3 "" H 2950 6300 60  0001 C CNN
 	1    2950 6300
 	1    0    0    -1
@@
 F 0 "#PWR?" H 2950 7150 30  0001 C CNN
 F 1 "GND" H 2950 7080 30  0001 C CNN
+F 2 "" H 2950 7150 60  0001 C CNN
+F 3 "" H 2950 7150 60  0001 C CNN
 	1    2950 7150
 	1    0    0    -1
@@
 F 0 "#PWR?" H 6750 5550 30  0001 C CNN
 F 1 "GND" H 6750 5480 30  0001 C CNN
+F 2 "" H 6750 5550 60  0001 C CNN
+F 3 "" H 6750 5550 60  0001 C CNN
 	1    6750 5550
 	1    0    0    -1
@@
 F 0 "SW?" H 3350 2400 50  0001 C CNN
 F 1 "Red E-Shutoff" H 3350 2250 50  0000 C CNN
+F 2 "" H 3350 2400 60  0001 C CNN
+F 3 "" H 3350 2400 60  0001 C CNN
 	1    3350 2400
 	1    0    0    -1
@@
 F 0 "K?" H 4285 7375 70  0001 C CNN
 F 1 "24vac_transformer" H 4535 6905 70  0001 C CNN
+F 2 "" H 4050 7250 60  0001 C CNN
+F 3 "" H 4050 7250 60  0001 C CNN
 	1    4050 7250
 	1    0    0    -1
 $EndComp
 $Comp
-L CIRCULATOR Grundfos
+L Circulator Grundfos
 U 1 1 523B1CF2
 P 2250 7350
 F 0 "Grundfos" H 2255 7360 60  0000 C CNN
 F 1 "Startup" H 2255 7455 60  0000 C CNN
+F 2 "" H 2250 7350 60  0001 C CNN
+F 3 "" H 2250 7350 60  0001 C CNN
 	1    2250 7350
 	0    -1   -1   0
@@
 F 0 "#PWR?" H 2300 2800 30  0001 C CNN
 F 1 "GND" H 2300 2730 30  0001 C CNN
+F 2 "" H 2300 2800 60  0001 C CNN
+F 3 "" H 2300 2800 60  0001 C CNN
 	1    2300 2800
 	1    0    0    -1
 $EndComp
 $Comp
-L +120VAC #PWR?
+L +120Vac #PWR?
 U 1 1 523B1BD1
 P 2300 2400
 F 0 "#PWR?" H 2300 2350 20  0001 C CNN
 F 1 "+120VAC" H 2300 2500 30  0000 C CNN
+F 2 "" H 2300 2400 60  0001 C CNN
+F 3 "" H 2300 2400 60  0001 C CNN
 	1    2300 2400
 	1    0    0    -1
@@
 F 0 "#PWR?" H 2750 5550 30  0001 C CNN
 F 1 "GND" H 2750 5480 30  0001 C CNN
+F 2 "" H 2750 5550 60  0001 C CNN
+F 3 "" H 2750 5550 60  0001 C CNN
 	1    2750 5550
 	1    0    0    -1
 $EndComp
 $Comp
-L AQUASTAT Aq?
+L Aquastat Aq?
 U 1 1 5236145B
 P 6000 6050
 F 0 "Aq?" H 5865 6160 60  0001 C CNN
 F 1 "AQUASTAT" H 5980 6255 60  0000 C CNN
+F 2 "" H 6000 6050 60  0001 C CNN
+F 3 "" H 6000 6050 60  0001 C CNN
 	1    6000 6050
 	-1   0    0    -1
@@
 F 0 "L?" H 5175 7070 60  0001 C CNN
 F 1 "LWC" H 4775 7075 60  0000 C CNN
+F 2 "" H 4550 6250 60  0001 C CNN
+F 3 "" H 4550 6250 60  0001 C CNN
 	1    4550 6250
 	1    0    0    -1
 $EndComp
 $Comp
-L CIRCULATOR Taco
+L Circulator Taco
 U 1 1 523613FF
 P 2250 6500
 F 0 "Taco" H 2255 6510 60  0000 C CNN
 F 1 "Primary Pump" H 2255 6605 60  0000 C CNN
+F 2 "" H 2250 6500 60  0001 C CNN
+F 3 "" H 2250 6500 60  0001 C CNN
 	1    2250 6500
 	0    -1   -1   0
 $EndComp
 $Comp
-L CIRCULATOR Taco
+L Circulator Taco
 U 1 1 523613FA
 P 7250 5300
 F 0 "Taco" H 7255 5310 60  0000 C CNN
 F 1 "Pool" H 7255 5405 60  0000 C CNN
+F 2 "" H 7250 5300 60  0001 C CNN
+F 3 "" H 7250 5300 60  0001 C CNN
 	1    7250 5300
 	0    1    1    0
@@
 F 0 "SW?" H 5600 1350 50  0000 C CNN
 F 1 "Pool Switch" H 5600 1050 50  0000 C CNN
+F 2 "" H 5600 1200 60  0001 C CNN
+F 3 "" H 5600 1200 60  0001 C CNN
 	1    5600 1200
 	1    0    0    -1
 $EndComp
 $Comp
-L ARGO A?
+L Argo A?
 U 1 1 523613D5
 P 4850 3150
 F 0 "A?" H 4975 4050 60  0001 C CNN
 F 1 "ARGO" H 5025 4175 60  0000 C CNN
+F 2 "" H 4850 3150 60  0001 C CNN
+F 3 "" H 4850 3150 60  0001 C CNN
 	1    4850 3150
 	1    0    0    -1
@@
 F 0 "E?" H 3500 6850 60  0001 C CNN
 F 1 "ECONOBURN" H 2950 6850 60  0000 C CNN
+F 2 "" H 2650 5550 60  0001 C CNN
+F 3 "" H 2650 5550 60  0001 C CNN
 	1    2650 5550
 	1    0    0    -1
