File: Interior.sch (KiCad schematic (older format))
At the start: 21 parts

Commit message: Generate PDFs
I opened this in the 4.0.2 version of kicad and it asked to make these changes.
Also included is the PDFs of the schematics.
Parts:
- Grundfos, Taco: symbol CIRCULATOR -> Circulator
- JC?: symbol PROBE -> Probe
- K?: symbol 24VAC_TRANSFORMER -> 24vac_transformer
- K? (x2): symbol 2PORT -> 2port
Changed lines of the file:
@@
-EESchema Schematic File Version 2  date Fri 20 Jun 2014 06:58:55 PM EDT
+EESchema Schematic File Version 2
+LIBS:Interior-rescue
 LIBS:power
 LIBS:device
@@
 LIBS:memory
 LIBS:xilinx
-LIBS:special
 LIBS:microcontrollers
 LIBS:dsp
@@
 LIBS:boiler
 LIBS:relay
-EELAYER 25  0
+EELAYER 25 0
 EELAYER END
-$Descr A4 11700 8267
+$Descr A4 11693 8268
 encoding utf-8
 Sheet 1 1
@@
 Wire Wire Line
 	3550 5700 3650 5700
-Connection ~ 8000 6450
-Wire Wire Line
-	7500 6450 8000 6450
-Wire Wire Line
-	8000 6450 9900 6450
-Wire Wire Line
-	3750 3350 3450 3350
-Wire Wire Line
-	3450 3350 2600 3350
+Connection ~ 8000 6350
+Wire Wire Line
+	7500 6350 8000 6350
+Wire Wire Line
+	8000 6350 9900 6350
+Wire Wire Line
+	2600 3350 3450 3350
+Wire Wire Line
+	3450 3350 3750 3350
 Wire Wire Line
 	1400 3200 1650 3200
@@
 	1300 4650 1300 4550
 Wire Wire Line
-	3700 4450 3700 4400
-Wire Wire Line
-	3700 4400 2900 4400
-Wire Wire Line
-	2900 4400 2500 4400
+	3700 4400 3700 4450
+Wire Wire Line
+	2500 4400 2900 4400
+Wire Wire Line
+	2900 4400 3700 4400
 Connection ~ 8000 5850
 Wire Wire Line
@@
 Connection ~ 9050 5850
 Wire Wire Line
-	8600 6100 9050 6100
-Wire Wire Line
-	9050 6100 9050 5850
-Wire Wire Line
-	9050 5850 9050 5650
+	9050 6100 8600 6100
+Wire Wire Line
+	9050 5650 9050 5850
+Wire Wire Line
+	9050 5850 9050 6100
 Wire Wire Line
 	2000 7100 2300 7100
@@
 	2300 7100 2700 7100
 Wire Wire Line
-	1800 7100 1550 7100
-Wire Wire Line
-	1550 7100 1000 7100
+	1000 7100 1550 7100
+Wire Wire Line
+	1550 7100 1800 7100
 Wire Wire Line
 	2700 7100 2700 7050
 Connection ~ 7650 3800
 Wire Wire Line
-	8350 3300 7550 3300
-Wire Wire Line
-	7550 3300 5900 3300
-Wire Wire Line
-	5900 3300 3850 3300
+	3850 3300 5900 3300
+Wire Wire Line
+	5900 3300 7550 3300
+Wire Wire Line
+	7550 3300 8350 3300
 Connection ~ 3450 3350
 Connection ~ 3750 3350
@@
 	10000 3800 8950 3800
 Wire Wire Line
-	7850 3800 7650 3800
-Wire Wire Line
-	7650 3800 7550 3800
+	7550 3800 7650 3800
+Wire Wire Line
+	7650 3800 7850 3800
 Wire Wire Line
 	7550 3800 7550 3650
@@
 	4100 3550 4100 3150
 Wire Wire Line
-	4100 3550 3350 3550
-Wire Wire Line
-	3350 3550 3350 3250
-Wire Wire Line
-	3350 3250 3350 3150
+	3350 3550 4100 3550
+Wire Wire Line
+	3350 3150 3350 3250
+Wire Wire Line
+	3350 3250 3350 3550
 Wire Wire Line
 	7550 3300 7550 3450
@@
 	9050 5650 8600 5650
 Wire Wire Line
-	8400 6100 8000 6100
-Wire Wire Line
-	8000 6100 8000 5850
-Wire Wire Line
-	8000 5850 8000 5650
+	8000 6100 8400 6100
+Wire Wire Line
+	8000 5650 8000 5850
+Wire Wire Line
+	8000 5850 8000 6100
 Wire Wire Line
 	8000 5650 8400 5650
 Wire Wire Line
-	9900 6450 9900 5850
-Wire Wire Line
-	2300 4400 2050 4400
-Wire Wire Line
-	2050 4400 1300 4400
+	9900 6350 9900 5850
+Wire Wire Line
+	1300 4400 2050 4400
+Wire Wire Line
+	2050 4400 2300 4400
 Wire Wire Line
 	1300 4400 1300 4450
@@
 	10300 5850 10300 5900
 Wire Wire Line
-	2800 7050 2800 7400
-Wire Wire Line
-	2800 7400 1550 7400
-Wire Wire Line
-	1550 7400 1000 7400
+	2800 7400 2800 7050
+Wire Wire Line
+	1000 7400 1550 7400
+Wire Wire Line
+	1550 7400 2800 7400
 Connection ~ 1550 7400
 Wire Wire Line
@@
 F 0 "K?" H 3468 5999 70  0001 C CNN
 F 1 "Thermostat2" H 3377 6121 70  0001 C CNN
+F 2 "" H 3300 5800 60  0001 C CNN
+F 3 "" H 3300 5800 60  0001 C CNN
 	1    3300 5800
 	1    0    0    -1
@@
 F 0 "K?" H 3868 5999 70  0001 C CNN
 F 1 "Thermostat2" H 3777 6121 70  0001 C CNN
+F 2 "" H 3700 5800 60  0001 C CNN
+F 3 "" H 3700 5800 60  0001 C CNN
 	1    3700 5800
 	1    0    0    -1
@@
 Text Notes 1000 7400 0    60   ~ 0
 White
-Text Notes 7500 6550 0    60   ~ 0
+Text Notes 6800 6400 0    60   ~ 0
 White\n(Smith Boiler)
 Text Notes 6050 4600 0    60   ~ 0
@@
 F 0 "#PWR?" H 1400 3450 30  0001 C CNN
 F 1 "GND" H 1400 3380 30  0001 C CNN
+F 2 "" H 1400 3450 60  0001 C CNN
+F 3 "" H 1400 3450 60  0001 C CNN
 	1    1400 3450
 	1    0    0    -1
 $EndComp
 $Comp
-L +120VAC #PWR?
+L +120Vac #PWR?
 U 1 1 523BC251
 P 1400 3200
 F 0 "#PWR?" H 1400 3150 20  0001 C CNN
 F 1 "+120VAC" H 1400 3300 30  0000 C CNN
+F 2 "" H 1400 3200 60  0001 C CNN
+F 3 "" H 1400 3200 60  0001 C CNN
 	1    1400 3200
 	1    0    0    -1
@@
 Black
 $Comp
-L CIRCULATOR Taco
+L Circulator Taco
 U 1 1 523B3663
 P 5400 6900
 F 0 "Taco" H 5405 6910 60  0000 C CNN
 F 1 "Basement" H 5405 7005 60  0000 C CNN
+F 2 "" H 5400 6900 60  0001 C CNN
+F 3 "" H 5400 6900 60  0001 C CNN
 	1    5400 6900
 	0    1    1    0
 $EndComp
 $Comp
-L CIRCULATOR Grundfos
+L Circulator Grundfos
 U 1 1 523B365D
 P 5400 6100
 F 0 "Grundfos" H 5405 6110 60  0000 C CNN
 F 1 "1st Floor" H 5405 6205 60  0000 C CNN
+F 2 "" H 5400 6100 60  0001 C CNN
+F 3 "" H 5400 6100 60  0001 C CNN
 	1    5400 6100
 	0    1    1    0
@@
 Text Notes 2500 7400 0    60   ~ 0
 White
-Text Notes 7250 5900 0    60   ~ 0
+Text Notes 6800 5900 0    60   ~ 0
 Red\n(Smith Boiler)\n
 Text Notes 9900 6000 0    60   ~ 0
@@
 Tripple \nAquastat \nRelay
 $Comp
-L 2PORT K?
+L 2port K?
 U 1 1 523B33FB
 P 3650 4500
 F 0 "K?" H 3818 4539 70  0001 C CNN
 F 1 "2PORT" H 3375 4551 70  0001 C CNN
+F 2 "" H 3650 4500 60  0001 C CNN
+F 3 "" H 3650 4500 60  0001 C CNN
 	1    3650 4500
 	0    1    1    0
 $EndComp
 $Comp
-L 2PORT K?
+L 2port K?
 U 1 1 523B33F4
 P 1350 4500
 F 0 "K?" H 1518 4539 70  0001 C CNN
 F 1 "2PORT" H 1075 4551 70  0001 C CNN
+F 2 "" H 1350 4500 60  0001 C CNN
+F 3 "" H 1350 4500 60  0001 C CNN
 	1    1350 4500
 	0    -1   -1   0
@@
 F 0 "R?" V 2748 4509 70  0001 C CNN
 F 1 "N/C" H 2397 4521 70  0000 C CNN
+F 2 "" H 2300 4400 60  0001 C CNN
+F 3 "" H 2300 4400 60  0001 C CNN
 F 4 "Relay" H 2348 4309 60  0000 C CNN "For"
 F 5 "1" H 2548 4309 60  0000 C CNN "Number"
@@
 F 0 "#PWR?" H 10300 5900 30  0001 C CNN
 F 1 "GND" H 10300 5830 30  0001 C CNN
+F 2 "" H 10300 5900 60  0001 C CNN
+F 3 "" H 10300 5900 60  0001 C CNN
 	1    10300 5900
 	1    0    0    -1
 $EndComp
 $Comp
-L +120VAC #PWR?
+L +120Vac #PWR?
 U 1 1 523B3383
 P 7500 5850
 F 0 "#PWR?" H 7500 5800 20  0001 C CNN
 F 1 "+120VAC" H 7500 5950 30  0000 C CNN
+F 2 "" H 7500 5850 60  0001 C CNN
+F 3 "" H 7500 5850 60  0001 C CNN
 	1    7500 5850
 	1    0    0    -1
@@
 F 0 "R?" V 8698 6159 70  0001 C CNN
 F 1 "N/O" H 8497 6221 70  0000 C CNN
+F 2 "" H 8400 6100 60  0001 C CNN
+F 3 "" H 8400 6100 60  0001 C CNN
 F 4 "Relay" H 8448 6009 60  0000 C CNN "For"
 F 5 "3" H 8648 6009 60  0000 C CNN "Number"
@@
 F 0 "R?" V 8698 5709 70  0001 C CNN
 F 1 "N/O" H 8497 5771 70  0000 C CNN
+F 2 "" H 8400 5650 60  0001 C CNN
+F 3 "" H 8400 5650 60  0001 C CNN
 F 4 "Relay" H 8448 5559 60  0000 C CNN "For"
 F 5 "2" H 8648 5559 60  0000 C CNN "Number"
@@
 $EndComp
 $Comp
-L CIRCULATOR Taco
+L Circulator Taco
 U 1 1 523B3356
 P 9900 5350
 F 0 "Taco" H 9905 5360 60  0000 C CNN
 F 1 "House Pump" H 9905 5455 60  0000 C CNN
+F 2 "" H 9900 5350 60  0001 C CNN
+F 3 "" H 9900 5350 60  0001 C CNN
 	1    9900 5350
 	1    0    0    -1
@@
 F 0 "R?" V 7998 3759 70  0001 C CNN
 F 1 "N/C" H 7647 3771 70  0000 C CNN
+F 2 "" H 7550 3650 60  0001 C CNN
+F 3 "" H 7550 3650 60  0001 C CNN
 F 4 "Relay" H 7598 3559 60  0000 C CNN "For"
 F 5 "3" H 7798 3559 60  0000 C CNN "Number"
@@
 F 0 "R?" H 7848 3909 70  0001 C CNN
 F 1 "N/O" H 7847 4121 70  0001 C CNN
+F 2 "" H 7850 3800 60  0001 C CNN
+F 3 "" H 7850 3800 60  0001 C CNN
 	1    7850 3800
 	1    0    0    -1
@@
 F 0 "R?" V 1998 7359 70  0001 C CNN
 F 1 "N/O" H 1900 7200 70  0000 C CNN
+F 2 "" H 1800 7100 60  0001 C CNN
+F 3 "" H 1800 7100 60  0001 C CNN
 F 4 "Relay" H 1850 7000 60  0000 C CNN "For"
 F 5 "1" H 2050 7000 60  0000 C CNN "Number"
@@
 $EndComp
 $Comp
-L +120VAC #PWR?
+L +120Vac #PWR?
 U 1 1 523B313A
 P 1000 7100
 F 0 "#PWR?" H 1000 7050 20  0001 C CNN
 F 1 "+120VAC" H 1000 7200 30  0000 C CNN
+F 2 "" H 1000 7100 60  0001 C CNN
+F 3 "" H 1000 7100 60  0001 C CNN
 	1    1000 7100
 	1    0    0    -1
@@
 F 0 "A?" H 2675 7950 60  0000 C CNN
 F 1 "Argo_2_x" H 2825 8075 60  0000 C CNN
+F 2 "" H 2550 7050 60  0001 C CNN
+F 3 "" H 2550 7050 60  0001 C CNN
 	1    2550 7050
 	1    0    0    -1
@@
 F 0 "RC?" H 9650 4400 60  0001 C CNN
 F 1 "RELAY_COIL" H 9500 4550 60  0001 C CNN
+F 2 "" H 8650 4350 60  0001 C CNN
+F 3 "" H 8650 4350 60  0001 C CNN
 F 4 "Relay" H 8650 4400 60  0000 C CNN "Name"
 F 5 "3" H 8650 4250 60  0000 C CNN "Number"
@@
 F 0 "RC?" H 9650 3850 60  0001 C CNN
 F 1 "RELAY_COIL" H 9500 4000 60  0001 C CNN
+F 2 "" H 8650 3800 60  0001 C CNN
+F 3 "" H 8650 3800 60  0001 C CNN
 F 4 "Relay" H 8650 3850 60  0000 C CNN "Name"
 F 5 "2" H 8650 3700 60  0000 C CNN "Number"
@@
 F 0 "RC?" H 9650 3350 60  0001 C CNN
 F 1 "RELAY_COIL" H 9500 3500 60  0001 C CNN
+F 2 "" H 8650 3300 60  0001 C CNN
+F 3 "" H 8650 3300 60  0001 C CNN
 F 4 "Relay" H 8650 3350 60  0000 C CNN "Name"
 F 5 "1" H 8650 3200 60  0000 C CNN "Number"
@@
 	1    0    0    -1
 $EndComp
-Text Notes 4350 3700 0    60   ~ 0
+Text Notes 4200 4050 0    60   ~ 0
 50 Degree\nFreeze Protection\nThermostat\n(Not Installed)
 $Comp
@@
 F 0 "K?" H 4618 3549 70  0001 C CNN
 F 1 "Thermostat2" H 4527 3671 70  0001 C CNN
+F 2 "" H 4450 3350 60  0001 C CNN
+F 3 "" H 4450 3350 60  0001 C CNN
 	1    4450 3350
 	-1   0    0    1
@@
 Green/Silver
 $Comp
-L PROBE JC?
+L Probe JC?
 U 1 1 523B21F9
 P 2050 2350
 F 0 "JC?" H 1150 2450 60  0000 C CNN
 F 1 "PROBE" H 1200 2600 60  0000 C CNN
+F 2 "" H 2050 2350 60  0001 C CNN
+F 3 "" H 2050 2350 60  0001 C CNN
 	1    2050 2350
 	1    0    0    -1
 $EndComp
 $Comp
-L 24VAC_TRANSFORMER K?
+L 24vac_transformer K?
 U 1 1 523B20A2
 P 1650 3200
 F 0 "K?" H 1885 3325 70  0001 C CNN
 F 1 "24VAC_TRANSFORMER" H 2135 2855 70  0001 C CNN
+F 2 "" H 1650 3200 60  0001 C CNN
+F 3 "" H 1650 3200 60  0001 C CNN
 	1    1650 3200
 	1    0    0    -1
@@
 F 0 "JC?" H 3900 4650 60  0000 C CNN
 F 1 "A419" H 3250 4650 60  0000 C CNN
+F 2 "" H 3100 3350 60  0001 C CNN
+F 3 "" H 3100 3350 60  0001 C CNN
 	1    3100 3350
 	1    0    0    -1
